File: pq-4.kicad_pcb (KiCad board)
At the start: 2 copper layers, 111 parts, among them IC1 M5218, IC2 M5218, IC3 M5218, IC4 M5218, IC5 M5218, J1 Conn_01x07_Male, J2 Conn_01x10_Male, Q1 2SK184-GR, Q2 2SC3378-GR, Q3 C2458-GR, Q4 C2458-GR, Q5 2SC3378-GR, Q6 2SC3378-GR, Q7 2SK118-Y, Q8 2SK118-Y, Q9 2SC3378-GR

Commit message: Minor improvements.
Connections:
- R31 pad 2: Net-(R31-Pad2) -> A
Changed lines of the file:
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@@
     (zones 0)
     (modules 111)
-    (nets 76)
+    (nets 75)
   )
   (page A4)
@@
   (net 72 "Net-(C28-Pad2)")
   (net 73 "Net-(D1-Pad1)")
-  (net 74 "Net-(R31-Pad2)")
-  (net 75 "Net-(D1-Pad2)")
+  (net 74 "Net-(D1-Pad2)")
   (net_class Default "This is the default net class."
     (clearance 0.2)
@@
     (add_net "Net-(OUT1-PadT)")
     (add_net "Net-(R26-Pad1)")
-    (add_net "Net-(R31-Pad2)")
     (add_net "Net-(R56-Pad1)")
     (add_net PRES2)
@@
       (net 12 "Net-(IC3-Pad2)"))
     (pad 2 thru_hole oval (at 5.08 0 90) (size 1.4 1.4) (drill 0.7) (layers *.Cu *.Mask)
-      (net 74 "Net-(R31-Pad2)"))
+      (net 18 A))
     (model ${KISYS3DMOD}/Resistor_THT.3dshapes/R_Axial_DIN0204_L3.6mm_D1.6mm_P5.08mm_Horizontal.wrl
       (at (xyz 0 0 0))
@@
       (net 73 "Net-(D1-Pad1)"))
     (pad 2 thru_hole oval (at 5.08 0) (size 2 2) (drill 1) (layers *.Cu *.Mask)
-      (net 75 "Net-(D1-Pad2)"))
+      (net 74 "Net-(D1-Pad2)"))
     (model ${KISYS3DMOD}/Diode_THT.3dshapes/D_T-1_P5.08mm_Horizontal.wrl
       (at (xyz 0 0 0))
