File: bypass_panel/bypass_panel.kicad_pcb (KiCad board)
At the start: 2 copper layers, 30 x 14 mm, 4 parts, among them J1 Conn_01x04_Male, J2 Conn_01x04_Male, SW1 SW_MEC_5G_LED

Commit message: Production version 2019.11.19.
Other:
- board text added: "2019.11.18"
- board text added: "github.com/mar0x/pq-4"
- board text removed: "2019.11.07"
- board text removed: "https://github.com/mar0x/pq-4"
Changed lines of the file:
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@@
       (outputformat 1)
       (mirror false)
-      (drillshape 1)
+      (drillshape 0)
       (scaleselection 1)
-      (outputdirectory ""))
+      (outputdirectory "gerber"))
   )
   (net 0 "")
@@
     (descr "Through hole straight pin header, 1x04, 2.54mm pitch, single row")
     (tags "Through hole pin header THT 1x04 2.54mm single row")
-    (fp_text reference J1 (at -2.54 -0.635 180) (layer B.SilkS)
+    (fp_text reference J1 (at -2.54 -0.635 180) (layer B.SilkS) hide
       (effects (font (size 1 1) (thickness 0.15)) (justify mirror))
     )
@@
     (descr "Through hole straight pin header, 1x04, 2.54mm pitch, single row")
     (tags "Through hole pin header THT 1x04 2.54mm single row")
-    (fp_text reference J2 (at -1.905 1.905) (layer B.SilkS)
+    (fp_text reference J2 (at -1.905 1.905) (layer B.SilkS) hide
       (effects (font (size 1 1) (thickness 0.15)) (justify mirror))
     )
@@
       (xy -2.9464 2.607733) (xy -2.9464 2.510946)) (layer B.SilkS) (width 0.01))
   )
-  (gr_text https://github.com/mar0x/pq-4 (at 144.145 86.995) (layer B.SilkS)
-    (effects (font (size 0.8 0.7) (thickness 0.15)) (justify mirror))
+  (gr_text github.com/mar0x/pq-4 (at 144.145 86.995) (layer B.SilkS)
+    (effects (font (size 0.7 0.8) (thickness 0.15)) (justify mirror))
   )
   (gr_text + (at 148.59 97.028) (layer F.SilkS)
@@
     (effects (font (size 1 1) (thickness 0.2)))
   )
-  (gr_text 2019.11.07 (at 139.7 97.79) (layer B.SilkS)
-    (effects (font (size 0.6 0.6) (thickness 0.1)) (justify mirror))
+  (gr_text 2019.11.18 (at 140.335 97.79) (layer B.SilkS)
+    (effects (font (size 0.9 0.9) (thickness 0.2)) (justify mirror))
   )
   (gr_line (start 147.32 92.71) (end 149.86 92.71) (layer F.SilkS) (width 0.2))
