File: digi_pot/digi_pot.sch (KiCad schematic (older format))
At the start: 22 parts, among them J1 Conn_01x08_Male, J2 Conn_01x06_Male, J3 Conn_01x03_Male, J4 Conn_01x03_Male, J5 Conn_01x06_Male, SW1 Rotary_Encoder, U1 ATmega328P-AU, U2 MCP42050

Commit message: Switching to AD5262 digital pot.
Parts:
- removed U2: MCP42050, Package_SO:TSSOP-14_4.4x5mm_P0.65mm, symbol Potentiometer_Digital:MCP42050
- added C4: 10u, Capacitor_Tantalum_SMD:CP_EIA-3216-18_Kemet-A_Pad1.58x1.35mm_HandSolder, symbol Device:CP_Small
- added C5: 0.1u, Capacitor_SMD:C_0805_2012Metric_Pad1.15x1.40mm_HandSolder, symbol Device:C_Small
- added J6: Conn_01x01_Male, Connector_PinHeader_2.54mm:PinHeader_1x01_P2.54mm_Vertical, symbol Connector:Conn_01x01_Male
- added U2: AD5262, Package_SO:TSSOP-16_4.4x5mm_P0.65mm, symbol ad5262:AD5262
- R10, R11, R5, R6, R7, R8, R9: value 10k -> 30k
- U1: symbol MCU_Microchip_ATmega:ATmega328P-AU -> digi_pot-rescue:ATmega328P-AU-MCU_Microchip_ATmega
Connections:
- net labels added: +9V
- wire segments 28 -> 41
- no-connect marks 0 -> 4
Other:
- moved on the sheet: J3, J4

Commit message: Using standard Atmega328 symbol.
Parts:
- removed U1: ATmega328P-AU, Package_QFP:TQFP-32_7x7mm_P0.8mm, symbol digi_pot-rescue:ATmega328P-AU-MCU_Microchip_ATmega
- added U1: ATmega328P-AU, Package_QFP:TQFP-32_7x7mm_P0.8mm, symbol MCU_Microchip_ATmega:ATmega328P-AU
Changed lines of the file:
@@
 $EndDescr
 $Comp
-L digi_pot-rescue:ATmega328P-AU-MCU_Microchip_ATmega U1
-U 1 1 601C4EF1
+L MCU_Microchip_ATmega:ATmega328P-AU U1
+U 1 1 5E465EF5
 P 4950 3550
-F 0 "U1" H 5350 2100 50  0000 C CNN
-F 1 "ATmega328P-AU" H 5500 2000 50  0000 C CNN
+F 0 "U1" H 4500 5050 50  0000 C CNN
+F 1 "ATmega328P-AU" H 5350 2050 50  0000 C CNN
 F 2 "Package_QFP:TQFP-32_7x7mm_P0.8mm" H 4950 3550 50  0001 C CIN
 F 3 "http://ww1.microchip.com/downloads/en/DeviceDoc/ATmega328_P%20AVR%20MCU%20with%20picoPower%20Technology%20Data%20Sheet%2040001984A.pdf" H 4950 3550 50  0001 C CNN
@@
 $EndComp
 $Comp
-L power:GND #PWR?
+L power:GND #PWR0106
 U 1 1 5E39246B
 P 7600 3250
-F 0 "#PWR?" H 7600 3000 50  0001 C CNN
+F 0 "#PWR0106" H 7600 3000 50  0001 C CNN
 F 1 "GND" H 7605 3077 50  0000 C CNN
 F 2 "" H 7600 3250 50  0001 C CNN
@@
 	7600 3250 7650 3250
 $Comp
-L power:+5V #PWR?
+L power:+5V #PWR0107
 U 1 1 5E39336E
 P 7650 2050
-F 0 "#PWR?" H 7650 1900 50  0001 C CNN
+F 0 "#PWR0107" H 7650 1900 50  0001 C CNN
 F 1 "+5V" H 7700 2200 50  0000 C CNN
 F 2 "" H 7650 2050 50  0001 C CNN
@@
 $EndComp
 $Comp
-L power:GND #PWR?
+L power:GND #PWR0116
 U 1 1 5E395ED2
 P 7050 3250
-F 0 "#PWR?" H 7050 3000 50  0001 C CNN
+F 0 "#PWR0116" H 7050 3000 50  0001 C CNN
 F 1 "GND" H 7055 3077 50  0000 C CNN
 F 2 "" H 7050 3250 50  0001 C CNN
@@
 NoConn ~ 7150 2750
 $Comp
-L power:+9V #PWR?
+L power:+9V #PWR0121
 U 1 1 5E3A4165
 P 7550 2050
-F 0 "#PWR?" H 7550 1900 50  0001 C CNN
+F 0 "#PWR0121" H 7550 1900 50  0001 C CNN
 F 1 "+9V" H 7450 2200 50  0000 C CNN
 F 2 "" H 7550 2050 50  0001 C CNN
@@
 $EndComp
 $Comp
-L power:+9V #PWR?
+L power:+9V #PWR0122
 U 1 1 5E3A5490
 P 6300 2050
-F 0 "#PWR?" H 6300 1900 50  0001 C CNN
+F 0 "#PWR0122" H 6300 1900 50  0001 C CNN
 F 1 "+9V" H 6200 2200 50  0000 C CNN
 F 2 "" H 6300 2050 50  0001 C CNN
@@
 $EndComp
 $Comp
-L power:GND #PWR?
+L power:GND #PWR0123
 U 1 1 5E3A5F6A
 P 6300 2350
-F 0 "#PWR?" H 6300 2100 50  0001 C CNN
+F 0 "#PWR0123" H 6300 2100 50  0001 C CNN
 F 1 "GND" H 6305 2177 50  0000 C CNN
 F 2 "" H 6300 2350 50  0001 C CNN
@@
 $EndComp
 $Comp
-L power:+9V #PWR?
+L power:+9V #PWR0124
 U 1 1 5E419DC4
 P 3600 5500
-F 0 "#PWR?" H 3600 5350 50  0001 C CNN
+F 0 "#PWR0124" H 3600 5350 50  0001 C CNN
 F 1 "+9V" H 3500 5650 50  0000 C CNN
 F 2 "" H 3600 5500 50  0001 C CNN
