File: pot_board/pot_board.kicad_pcb (KiCad board)
At the start: 2 copper layers, 33 parts, among them J1 ISCP, J2 Conn_01x07_Pin, J3 Conn_01x10_Pin, J4 Conn_01x05_Pin, U1 ATmega328P-A, U3 AD5262, U4 AD5262, U5 AD5262, U6 AD5262, U7 AD5262, U8 AD5262, U9 AD5262

Commit message: Working on POT Board
Parts:
- added C20: 10uF, Capacitor_THT:CP_Radial_D4.0mm_P2.00mm, F.Cu at (147.9, 35.7)
- added C21: 10uF, Capacitor_THT:CP_Radial_D4.0mm_P2.00mm, F.Cu at (147.9, 47.1)
- added C22: 10uF, Capacitor_THT:CP_Radial_D4.0mm_P2.00mm, F.Cu at (148.1, 58.5)
- added C23: 10uF, Capacitor_THT:CP_Radial_D4.0mm_P2.00mm, F.Cu at (177.9, 134.6)
- added C24: 10uF, Capacitor_THT:CP_Radial_D4.0mm_P2.00mm, F.Cu at (177.8, 149.9)
- added C25: 10uF, Capacitor_THT:CP_Radial_D4.0mm_P2.00mm, F.Cu at (175.8, 165.1)
- added C26: 10uF, Capacitor_THT:CP_Radial_D4.0mm_P2.00mm, F.Cu at (137.7, 149.9)
- added C4: 10uF, Capacitor_THT:CP_Radial_D4.0mm_P2.00mm, F.Cu at (178.7, 92.7)
- added C5: 47uF, Capacitor_THT:CP_Radial_D4.0mm_P2.00mm, F.Cu at (178.7, 102.2)
- J2: value Conn_01x07_Pin -> PQ-4A; moved to B.Cu
- J3: value Conn_01x10_Pin -> PQ-4B; moved to B.Cu
- J4: value Conn_01x05_Pin -> I2C_control
- moved C18 88.9 mm to (171.8, 167.6)
- moved C11 85.3 mm to (171.8, 162.6)
- moved C17 77.1 mm to (171.8, 152.4)
- moved C10 74.1 mm to (172.7, 147.3)
- moved C19 69.4 mm to (133.7, 152.4)
- moved C12 63.4 mm to (134.6, 147.3)
- moved U8 60.5 mm to (165.1, 165.1)
- moved U7 53.3 mm to (165.1, 149.9)
- moved C6 53.0 mm to (161.1, 39.1), turned to -90 degrees
- moved J4 51.6 mm to (106.3, 99.1)
- moved C16 51.3 mm to (172.7, 139.7)
- moved C27 50.9 mm to (114.7, 50.2)
- moved J1 49.7 mm to (101.6, 83.8)
- moved C9 49.3 mm to (171.8, 134.6)
- moved C13 48.5 mm to (147.9, 39.3), turned to -90 degrees
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